File: ProtocolPro/ProtocolPro.kicad_sch (KiCad schematic)
At the start: 8 parts, among them J1 CAN Bus Splitter, U2 TBA1-0512E, U3 TBA1-0512E

Commit message: added more components
Parts:
- added J1: Conn_01x04, symbol Connector_Generic:Conn_01x04
Connections:
- net at BRD1. (CAN2): now also J1.5 (Pin_5)
- new net: BRD1. (CAN2), U1. (VCC_5V) (x5)
- new net 5V: J1.4 (Pin_4)
- new net GND: J1.3 (Pin_3)
- new net RX: J1.1 (Pin_1)
- new net TX: J1.2 (Pin_2)
Other:
- note added: "For RX receiver"
Changed lines of the file:
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@@
+		)
+	)
+	(text "For RX receiver"
+		(exclude_from_sim no)
+		(at 68.834 84.582 0)
+		(effects
+			(font
+				(size 1.27 1.27)
+			)
 		)
 	)
@@
 		)
 	)
+	(label "GND"
+		(at 63.5 77.47 0)
+		(effects
+			(font
+				(size 1.27 1.27)
+			)
+			(justify left bottom)
+		)
+	)
+	(label "RX"
+		(at 63.5 82.55 0)
+		(effects
+			(font
+				(size 1.27 1.27)
+			)
+			(justify left bottom)
+		)
+	)
+	(label "TX"
+		(at 63.5 80.01 0)
+		(effects
+			(font
+				(size 1.27 1.27)
+			)
+			(justify left bottom)
+		)
+	)
+	(label "5V"
+		(at 63.5 74.93 0)
+		(effects
+			(font
+				(size 1.27 1.27)
+			)
+			(justify left bottom)
+		)
+	)
+	(symbol
+		(lib_id "Connector_Generic:Conn_01x04")
+		(at 58.42 80.01 180)
+		(unit 1)
+		(exclude_from_sim no)
+		(in_bom yes)
+		(on_board yes)
+		(dnp no)
+		(fields_autoplaced yes)
+		(property "Reference" "J1"
+			(at 58.42 68.58 0)
+			(effects
+				(font
+					(size 1.27 1.27)
+				)
+			)
+		)
+		(property "Value" "Conn_01x04"
+			(at 58.42 71.12 0)
+			(effects
+				(font
+					(size 1.27 1.27)
+				)
+			)
+		)
+		(property "Footprint" ""
+			(at 58.42 80.01 0)
+			(effects
+				(font
+					(size 1.27 1.27)
+				)
+				(hide yes)
+			)
+		)
+		(property "Datasheet" "~"
+			(at 58.42 80.01 0)
+			(effects
+				(font
+					(size 1.27 1.27)
+				)
+				(hide yes)
+			)
+		)
+		(property "Description" "Generic connector, single row, 01x04, script generated (kicad-library-utils/schlib/autogen/connector/)"
+			(at 58.42 80.01 0)
+			(effects
+				(font
+					(size 1.27 1.27)
+				)
+				(hide yes)
+			)
+		)
+		(pin "2"
+		)
+		(pin "1"
+		)
+		(pin "4"
+		)
+		(pin "3"
+		)
+		(instances
+			(project ""
+				(path "/90d848c3-1c3b-483b-a276-b23aa2b65688"
+					(reference "J1")
+					(unit 1)
+				)
+			)
+		)
+	)

Commit message: draft 1 ready
Parts:
- removed J1: Conn_01x04, symbol Connector_Generic:Conn_01x04
- removed J1: CAN Bus Splitter, symbol Connector_Generic:Conn_01x05
- removed U2, U3: TBA1-0512E, Converter_DCDC:Converter_DCDC_TRACO_TBA1-xxxxE_Single_THT, symbol Converter_DCDC:TBA1-0512E
- added U?: LIS3MDL, Package_LGA:LGA-12_2x2mm_P0.5mm, symbol Sensor_Magnetic:LIS3MDL
- added U?: Happymodel EP1, symbol ProtocolProCustomSymbols:Happymodel_EP1
Connections:
- net GND: now also BRD1. (CAN2), U1. (VCC_5V), U?.1 (GND), U?.12 (GND), U?.18 (GND), U?.3 (GND), U?.7 (GND), U?.12 (GND), U?.2 (GND), U?.3 (GND)
- net VCC: now reaches BRD1. (CAN2)
- net VCC: now also U1. (VCC_5V), U?.13 (VDD), U?.4 (VCC), U?.8 (VDD), U?.5 (Vdd)
- net at U?.1 (RXD1): now also BRD1. (CAN2), U?.2 (TXD1)
- net I2C2: now reaches U?.23 (SCL)
- net I2C2: now also BRD1. (CAN2), U?.2 (CSB), U?.24 (SDA), U?.3 (SDI), U?.4 (SCK), U?.5 (SDO), U?.11 (SDA/SDI/SDO), U?.9 (SDO/SA1)
- new net: BRD1. (CAN2), U?. (RX)
- new net: BRD1. (CAN2), U1. (VCC_5V) (x4)
- no-connect marks 0 -> 39
Other:
- note added: "Magnetometer"
- note removed: "5.3v step down module"
- note removed: "For RX receiver"
- note removed: "To add: battery, rx tx, gimbal + camera"
- moved on the sheet: U1, U?
